Commit message: fixed urdf file paths to stl file

File: src/viz/models/biomimic_hand_v3/urdf/biomimic_hand.urdf (robot description, URDF)
Before this commit: robot converted_robot, 99 links, 98 joints
Links:
- link index_abduct_link: geometry visual mesh filename=package://viz/models/biomimic_hand_v3/mesh/experimental_fin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
- link index_base: geometry visual mesh filename=package://viz/models/biomimic_hand_v3/mesh/experimental_fin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
- link index_dp_adapter: geometry visual mesh filename=package://viz/models/biomimic_hand_v3/mesh/experimental_fin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
- link index_mp_link: geometry visual mesh filename=package://viz/models/biomimic_hand_v3/mesh/experimental_fin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
- link index_pp_link: geometry visual mesh filename=package://viz/models/biomimic_hand_v3/mesh/experimental_fin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
- link middle_abduct_link: geometry visual mesh filename=package://viz/models/biomimic_hand_v3/mesh/experimental_fin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
- link middle_base: geometry visual mesh filename=package://viz/models/biomimic_hand_v3/mesh/experimental_fin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
- link middle_dp_adapter: geometry visual mesh filename=package://viz/models/biomimic_hand_v3/mesh/experimental_fin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
- link middle_mp_link: geometry visual mesh filename=package://viz/models/biomimic_hand_v3/mesh/experimental_fin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
- link middle_pp_link: geometry visual mesh filename=package://viz/models/biomimic_hand_v3/mesh/experimental_fin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
- link palm: geometry visual mesh filename=package://viz/models/biomimic_hand_v3/mesh/Wrist_Counterpar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; visual mesh filename=package://viz/models/biomimic_hand_v3/mesh/palm_reframed.stl
- link pinky_abduct_link: geometry visual mesh filename=package://viz/models/biomimic_hand_v3/mesh/experimental_fin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
- link pinky_base: geometry visual mesh filename=package://viz/models/biomimic_hand_v3/mesh/experimental_fin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
- link pinky_dp_adapter: geometry visual mesh filename=package://viz/models/biomimic_hand_v3/mesh/experimental_fin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
- link pinky_mp_link: geometry visual mesh filename=package://viz/models/biomimic_hand_v3/mesh/experimental_fin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
- link pinky_pp_link: geometry visual mesh filename=package://viz/models/biomimic_hand_v3/mesh/experimental_fin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
- link ring_abduct_link: geometry visual mesh filename=package://viz/models/biomimic_hand_v3/mesh/experimental_fin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
- link ring_base: geometry visual mesh filename=package://viz/models/biomimic_hand_v3/mesh/experimental_fin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
- link ring_dp_adapter: geometry visual mesh filename=package://viz/models/biomimic_hand_v3/mesh/experimental_fin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
- link ring_mp_link: geometry visual mesh filename=package://viz/models/biomimic_hand_v3/mesh/experimental_fin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
- link ring_pp_link: geometry visual mesh filename=package://viz/models/biomimic_hand_v3/mesh/experimental_fin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
- link root: geometry visual mesh filename=package://viz/models/biomimic_hand_v3/mesh/Tower_reframed.s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; visual mesh filename=package://viz/models/biomimic_hand_v3/mesh/Wrist_concept_ac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
- link thumb_base: geometry visual mesh filename=package://viz/models/biomimic_hand_v3/mesh/thumb_base_refra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
- link thumb_dp: geometry visual mesh filename=package://viz/models/biomimic_hand_v3/mesh/thumb_tip.stl
- link thumb_mp: geometry visual mesh filename=package://viz/models/biomimic_hand_v3/mesh/thumb_link_3_ref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
- link thumb_pp: geometry visual mesh filename=package://viz/models/biomimic_hand_v3/mesh/thumb_link2_refr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
