Commit message: full pipeline with retarget & rosbag integration, only handcontroller missing now

File: src/viz/models/orca1_hand/urdf/orca1.urdf (robot description, URDF)
Before this commit: robot converted_robot, 53 links, 52 joints
Links:
- removed link world
- removed link world2palm_fixed_jointbody
- added link hand_root, mass 0.0
- added link root2palm_fixed_jointbody, mass 0.001
- link index_dp: geometry visual mesh filename=package://viz/models/orca1_hand/urdf/converted_index_dp.stl
- link index_mp: geometry visual mesh filename=package://viz/models/orca1_hand/urdf/converted_index_mp.stl
- link index_pp: geometry visual mesh filename=package://viz/models/orca1_hand/urdf/converted_index_pp.stl
- link index_um: geometry visual mesh filename=package://viz/models/orca1_hand/urdf/converted_index_um.stl
- link middle_dp: geometry visual mesh filename=package://viz/models/orca1_hand/urdf/converted_middle_dp.stl
- link middle_mp: geometry visual mesh filename=package://viz/models/orca1_hand/urdf/converted_middle_mp.stl
- link middle_pp: geometry visual mesh filename=package://viz/models/orca1_hand/urdf/converted_middle_pp.stl
- link middle_um: geometry visual mesh filename=package://viz/models/orca1_hand/urdf/converted_middle_um.stl
- link palm: geometry visual mesh filename=package://viz/models/orca1_hand/urdf/converted_palm_tower.s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
- link pinky_dp: geometry visual mesh filename=package://viz/models/orca1_hand/urdf/converted_pinky_dp.stl
- link pinky_mp: geometry visual mesh filename=package://viz/models/orca1_hand/urdf/converted_pinky_mp.stl
- link pinky_pp: geometry visual mesh filename=package://viz/models/orca1_hand/urdf/converted_pinky_pp.stl
- link pinky_um: geometry visual mesh filename=package://viz/models/orca1_hand/urdf/converted_pinky_um.stl
- link ring_dp: geometry visual mesh filename=package://viz/models/orca1_hand/urdf/converted_ring_dp.stl
- link ring_mp: geometry visual mesh filename=package://viz/models/orca1_hand/urdf/converted_ring_mp.stl
- link ring_pp: geometry visual mesh filename=package://viz/models/orca1_hand/urdf/converted_ring_pp.stl
- link ring_um: geometry visual mesh filename=package://viz/models/orca1_hand/urdf/converted_ring_um.stl
- link thumb_base: geometry visual mesh filename=package://viz/models/orca1_hand/urdf/converted_thumb_base.s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
- link thumb_dp: geometry visual mesh filename=package://viz/models/orca1_hand/urdf/converted_thumb_dp.stl
- link thumb_mp: geometry visual mesh filename=package://viz/models/orca1_hand/urdf/converted_thumb_mp.stl
- link thumb_pp: geometry visual mesh filename=package://viz/models/orca1_hand/urdf/converted_thumb_pp.stl
Joints:
- removed joint world2palm_fixed
- removed joint world2palm_fixed_offset
- added joint root2palm_fixed: type fixed, parent hand_root, child root2palm_fixed_jointbody, origin xyz=0.0 0.0 0.0 rpy=0.0 0.0 0.0
- added joint root2palm_fixed_offset: type fixed, parent root2palm_fixed_jointbody, child palm, origin xyz=-0.0 -0.0 -0.0 rpy=0.0 0.0 0.0
- joint index_dp2index_fingertip_fixed: origin xyz=0.0 0.0 0.0 rpy=0.0 0.0 0.0 -> xyz=0.0 0.020 -0.001306 rpy=0.0 0.0 0.0
- joint middle_dp2middle_fingertip_fixed: origin xyz=0.0 0.0 0.0 rpy=0.0 0.0 0.0 -> xyz=0.0 0.020 -0.001306 rpy=0.0 0.0 0.0
- joint pinky_dp2pinky_fingertip_fixed: origin xyz=0.0 0.0 0.0 rpy=0.0 0.0 0.0 -> xyz=0.0 0.020 -0.001306 rpy=0.0 0.0 0.0
- joint ring_dp2ring_fingertip_fixed: origin xyz=0.0 0.0 0.0 rpy=0.0 0.0 0.0 -> xyz=0.0 0.020 -0.001306 rpy=0.0 0.0 0.0
- joint thumb_dp2thumb_fingertip_fixed: origin xyz=0.0 0.0 0.0 rpy=0.0 0.0 0.0 -> xyz=0.0 0.02425 -0.001189 rpy=0.0 0.0 0.0

Commit message: orca2.1: urdf file update with skin

File: src/viz/models/orca1_hand/urdf/orca1.urdf (robot description, URDF)
Before this commit: robot converted_robot, 53 links, 52 joints
Links:
- removed link hand_root
- added link root, mass 0.0
- added link world, mass 0.0
- added link world2root_fixed_jointbody, mass 0.001
- link index_dp: mass 0.0011385821737687244 -> 0.009142007854382036
- link index_mp: mass 0.003108373341414378 -> 0.007256911934241935
- link index_pp: mass 0.006075709241757069 -> 0.01253208205763138
- link middle_dp: mass 0.0011385821737687244 -> 0.009142007854382036
- link middle_mp: mass 0.003108373341414378 -> 0.007256911934241935
- link middle_pp: mass 0.007199054377400034 -> 0.015838995744240178
- link pinky_dp: mass 0.0011385821737687244 -> 0.009142007854382036
- link pinky_mp: mass 0.003108373341414378 -> 0.007256911934241935
- link pinky_pp: mass 0.0046751560406718806 -> 0.009193689280540233
- link ring_dp: mass 0.0011385821737687244 -> 0.009142007854382036
- link ring_mp: mass 0.003108373341414378 -> 0.007256911934241935
- link ring_pp: mass 0.007199054377400034 -> 0.015838995744240178
- link thumb_dp: mass 0.001814128231283667 -> 0.009142007854382036
Joints:
- added joint world2root_fixed: type fixed, parent world, child world2root_fixed_jointbody, origin xyz=0.0 0.0 0.0 rpy=0.0 0.0 0.0
- added joint world2root_fixed_offset: type fixed, parent world2root_fixed_jointbody, child root, origin xyz=-0.0 -0.0 -0.0 rpy=0.0 0.0 0.0
- joint index_abd: axis -5.551115123125783e-17 1.2212453270876722e-15 0.9999999999999968 -> -1.80855330711438e-13 -2.220446049250313e-16 0.9999999999999967; origin xyz=-0.0220268982915701 0.0015684105070722626 0.03555822504310243 rpy=1.6579894511737647 1.3961154673834115 -7.447055239240274e-05 -> xyz=-0.022026898291690793 0.0015684105070722376 0.035558225043043304 rpy=1.657989451174792 1.3961154673834115 -7.447055134812697e-05
- joint index_abd_offset: origin xyz=-0.014399999999999956 1.0278236595162582e-16 -1.431146867680866e-17 rpy=0.0 0.0 0.0 -> xyz=-0.014399999999999979 -1.1275702593849246e-17 -4.7704895589362195e-18 rpy=0.0 0.0 0.0
- joint index_mp2dp: axis -0.9999999999999996 -2.0261570199409107e-15 1.0547118733938987e-15 -> -0.9999999999999998 -1.1796119636642288e-16 -1.946657895643411e-15; origin xyz=0.0009999999999999543 -8.177594885971917e-17 0.027999999999999962 rpy=1.570796326794896 1.1102230246251565e-15 1.5707963267948963 -> xyz=0.0009999999999999601 -4.683753385137379e-17 0.028000000000000004 rpy=-6.661338147750939e-16 8.881784197001252e-16 1.5707963267948974
- joint index_mp2dp_offset: origin xyz=-9.999999999994138e-05 5.371544138307871e-17 3.0201383250825706e-17 rpy=0.0 0.0 0.0 -> xyz=-0.01099999999999995 7.281470469246501e-06 0.009007281470469294 rpy=0.0 0.0 0.0
- joint index_pp2mp: axis 8.326672684688674e-16 -0.9999999999999992 -9.506284648352903e-16 -> 1.0547118733938987e-15 -0.9999999999999989 -9.020562075079397e-16; origin xyz=-3.5654192458018814e-17 -1.9773193420734087e-17 0.04000000000000007 rpy=-6.938893903907228e-17 2.220446049250313e-16 1.1102230246251565e-16 -> xyz=-4.092895317840004e-17 -2.263553056912248e-17 0.039999999999999904 rpy=-1.387778780781445e-17 -2.220446049250313e-16 2.311115933264683e-33
- joint index_pp2mp_offset: origin xyz=1.722275552576525e-17 2.4110002110676104e-17 -3.2175644141916336e-17 rpy=0.0 0.0 0.0 -> xyz=1.9461750163187066e-17 3.195966925249782e-17 5.1027793401258624e-17 rpy=0.0 0.0 0.0
- joint middle_mp2dp: axis -0.9999999999999994 1.159735553967606e-16 6.744138602805412e-17 -> -1.0000000000000002 -3.2838929933875956e-17 5.315090385248316e-16; origin xyz=0.0010000000000000631 9.161508357502633e-18 0.028000000000000025 rpy=1.5707963267948948 0.0 1.5707963267948966 -> xyz=0.0010000000000037676 -2.2551405187698492e-17 0.027999999999999955 rpy=4.551914400963142e-14 -4.440892098500626e-16 1.5707963267948966
- joint middle_mp2dp_offset: origin xyz=-1.5612511283791412e-17 1.3361333028928368e-19 -1.2273161319545561e-16 rpy=0.0 0.0 0.0 -> xyz=-0.011000000000000034 7.28147046937894e-06 0.009007281470469267 rpy=0.0 0.0 0.0
- joint pinky_mp2dp: axis -1.0000000000000002 -3.0531133177191805e-16 -7.355227538141662e-16 -> -0.9999999999999996 2.3037127760972e-15 1.584097436557741e-13; origin xyz=0.0009999999999999842 6.46455545344482e-18 0.028000000000000067 rpy=1.570796326794896 4.440892098500626e-16 1.5707963267948968 -> xyz=0.0010000000000103548 -1.148039996401451e-14 0.02799999999999978 rpy=1.7696955012524995e-13 -1.5853984791647235e-13 1.5707963267948981
- joint pinky_mp2dp_offset: origin xyz=-0.00010000000000001497 -7.207742161365743e-17 -2.9290399316053706e-18 rpy=0.0 0.0 0.0 -> xyz=-0.011000000000000044 7.281470469290411e-06 0.00900728147046922 rpy=0.0 0.0 0.0
- joint ring_abd: axis 6.38378239159465e-16 7.771561172376096e-16 0.9999999999999978 -> -8.004708007547379e-14 -1.9984014443252818e-14 0.9999999999999978; origin xyz=0.019694864162417412 0.0013825982229840389 0.030586364349873878 rpy=-1.5707963267948921 1.3088618425821554 -3.054326190990074 -> xyz=0.019694864162417412 0.0013825982229840321 0.030586364349873787 rpy=-1.5707963267948921 1.3088618425821554 -3.054326190990074
- joint ring_abd_offset: origin xyz=-0.014399999999999944 5.941427905220564e-17 1.5178830414797062e-17 rpy=0.0 0.0 0.0 -> xyz=-0.014400000000000029 3.5561831257524545e-17 8.239936510889834e-18 rpy=0.0 0.0 0.0
- joint ring_mp2dp: axis -1.0000000000000004 -8.881784197001252e-16 9.020562075079397e-17 -> -1.0000000000000004 9.71445146547012e-17 4.7009379895712744e-15; origin xyz=0.0010000000000000406 1.4632114375292307e-16 0.028000000000000025 rpy=1.5707963267948963 2.6645352591003757e-15 1.5707963267948963 -> xyz=0.0010000000000000247 1.5785983631388945e-16 0.02800000000000006 rpy=-1.4432899320127035e-15 -2.886579864025407e-15 1.570796326794897
- joint ring_mp2dp_offset: origin xyz=-1.3721384550404466e-16 -6.547177265705249e-17 -4.2773936368871135e-17 rpy=0.0 0.0 0.0 -> xyz=-0.011000000000000136 7.2814704693049395e-06 0.009007281470469263 rpy=0.0 0.0 0.0
- joint ring_pp2mp: axis -2.7755575615628914e-16 -0.9999999999999994 1.734723475976807e-15 -> 5.551115123125783e-17 -0.9999999999999998 1.6514567491299204e-15; origin xyz=-8.020486901317957e-19 8.994390474632575e-17 0.04800000000000009 rpy=-2.465190328815662e-32 -4.440892098500626e-16 1.1102230246251565e-16 -> xyz=1.6557794334752767e-17 1.0283099349852077e-16 0.048000000000000105 rpy=-8.326672684688684e-17 4.440892098500626e-16 -4.440892098500627e-16
- joint ring_pp2mp_offset: origin xyz=-2.4785122580526127e-17 -9.905120299520399e-17 -1.2157278934836427e-17 rpy=0.0 0.0 0.0 -> xyz=-2.4797730845642552e-17 -9.545841872561936e-17 -2.5561932479781495e-17 rpy=0.0 0.0 0.0
- joint root2index_pp: axis 9.992007221626409e-16 -1.000000000000004 -1.0130785099704553e-15 -> 3.175237850427948e-14 -1.0000000000000018 -2.0646956366832114e-12; origin xyz=-6.511929505797567e-17 -1.2884579059542108e-16 1.2330918261215923e-17 rpy=-3.14159265358971 -1.5689140977438238 3.141592653589709 -> xyz=-3.726525911802163e-14 1.5826592868386048e-13 -1.3897728001093473e-14 rpy=3.141592653571369 -1.568914097743692 -3.1415926535734324
- joint root2index_pp_offset: origin xyz=-2.2103198581084714e-18 -7.053339437169385e-18 1.2080891234349761e-18 rpy=0.0 0.0 0.0 -> xyz=9.357535447968366e-19 9.360525909273759e-18 1.2460153634354755e-17 rpy=0.0 0.0 0.0
- joint root2palm_fixed: parent hand_root -> root
- joint root2ring_pp: axis -5.551115123125783e-17 -1.0000000000000022 1.7139067942650854e-15 -> 2.1538326677728037e-14 -1.0000000000000016 9.536885170469134e-13; origin xyz=-8.061277083623726e-17 -2.084317473075087e-17 -8.48575991563069e-18 rpy=3.1415926535897474 -1.569095233503671 -3.1415926535897465 -> xyz=8.76421389591046e-16 -6.591883351625457e-14 -5.609920274269105e-15 rpy=3.1415926535778085 -1.5690952335036443 -3.1415926535768572
- joint root2ring_pp_offset: origin xyz=2.763004548120401e-19 6.477168015932836e-18 1.61034059853451e-17 rpy=0.0 0.0 0.0 -> xyz=-9.795286269233676e-19 -1.4465518891423126e-19 1.4329772049885697e-17 rpy=0.0 0.0 0.0
- joint thumb_mp2dp: axis 0.9999999999999958 -9.992007221626409e-16 1.7486012637846216e-15 -> -0.9999999999999958 2.9976021664879227e-15 5.287437154777308e-15; limit lower=-1.7453292519943295 upper=0.0 effort=100 velocity=100 -> lower=0.0 upper=1.57 effort=100 velocity=100; origin xyz=1.239088163743751e-16 5.408958416957225e-16 0.03000000000000005 rpy=1.5707963267949039 -8.659739592076221e-15 1.570796326794891 -> xyz=1.8258726914308424e-16 5.204170427930421e-16 0.029999999999999895 rpy=2.4424906541753444e-15 -1.2878587085651816e-14 1.5707963267948923
- joint thumb_mp2dp_offset: origin xyz=-6.3846885802101e-17 -2.638575629691531e-17 -2.8715865630147274e-17 rpy=0.0 0.0 0.0 -> xyz=-0.011000000000000175 7.281470469432116e-06 0.009007281470469333 rpy=0.0 0.0 0.0

File: src/viz/models/orca2_hand/urdf/orca2.urdf (robot description, URDF)
Before this commit: robot converted_robot, 55 links, 54 joints
Links:
- removed link hand_root
- added link root, mass 0.0
- added link world, mass 0.0
- added link world2root_fixed_jointbody, mass 0.001
- link index_dp: mass 0.0011385821737687244 -> 0.009142007854382036
- link index_mp: mass 0.003108373341414378 -> 0.007256911934241935
- link index_pp: mass 0.006075709241757069 -> 0.01253208205763138
- link middle_dp: mass 0.0011385821737687244 -> 0.009142007854382036
- link middle_mp: mass 0.003108373341414378 -> 0.007256911934241935
- link middle_pp: mass 0.007199054377400034 -> 0.015838995744240178
- link pinky_dp: mass 0.0011385821737687244 -> 0.009142007854382036
- link pinky_mp: mass 0.003108373341414378 -> 0.007256911934241935
- link pinky_pp: mass 0.0046751560406718806 -> 0.009193689280540233
- link ring_dp: mass 0.0011385821737687244 -> 0.009142007854382036
- link ring_mp: mass 0.003108373341414378 -> 0.007256911934241935
- link ring_pp: mass 0.007199054377400034 -> 0.015838995744240178
- link thumb_dp: mass 0.001814128231283667 -> 0.009142007854382036
Joints:
- added joint world2root_fixed: type fixed, parent world, child world2root_fixed_jointbody, origin xyz=0.0 0.0 0.0 rpy=0.0 0.0 0.0
- added joint world2root_fixed_offset: type fixed, parent world2root_fixed_jointbody, child root, origin xyz=-0.0 -0.0 -0.0 rpy=0.0 0.0 0.0
- joint index_abd: axis -5.551115123125783e-17 1.2212453270876722e-15 0.9999999999999968 -> -1.80855330711438e-13 -2.220446049250313e-16 0.9999999999999967; origin xyz=-0.0220268982915701 0.0015684105070722626 0.03555822504310243 rpy=1.6579894511737647 1.3961154673834115 -7.447055239240274e-05 -> xyz=-0.022026898291690793 0.0015684105070722376 0.035558225043043304 rpy=1.657989451174792 1.3961154673834115 -7.447055134812697e-05
- joint index_abd_offset: origin xyz=-0.014399999999999956 1.0278236595162582e-16 -1.431146867680866e-17 rpy=0.0 0.0 0.0 -> xyz=-0.014399999999999979 -1.1275702593849246e-17 -4.7704895589362195e-18 rpy=0.0 0.0 0.0
- joint index_mp2dp: axis -0.9999999999999996 -2.0261570199409107e-15 1.0547118733938987e-15 -> -0.9999999999999998 -1.1796119636642288e-16 -1.946657895643411e-15; origin xyz=0.0009999999999999543 -8.177594885971917e-17 0.027999999999999962 rpy=1.570796326794896 1.1102230246251565e-15 1.5707963267948963 -> xyz=0.0009999999999999601 -4.683753385137379e-17 0.028000000000000004 rpy=-6.661338147750939e-16 8.881784197001252e-16 1.5707963267948974
- joint index_mp2dp_offset: origin xyz=-9.999999999994138e-05 5.371544138307871e-17 3.0201383250825706e-17 rpy=0.0 0.0 0.0 -> xyz=-0.01099999999999995 7.281470469246501e-06 0.009007281470469294 rpy=0.0 0.0 0.0
- joint index_pp2mp: axis 8.326672684688674e-16 -0.9999999999999992 -9.506284648352903e-16 -> 1.0547118733938987e-15 -0.9999999999999989 -9.020562075079397e-16; origin xyz=-3.5654192458018814e-17 -1.9773193420734087e-17 0.04000000000000007 rpy=-6.938893903907228e-17 2.220446049250313e-16 1.1102230246251565e-16 -> xyz=-4.092895317840004e-17 -2.263553056912248e-17 0.039999999999999904 rpy=-1.387778780781445e-17 -2.220446049250313e-16 2.311115933264683e-33
- joint index_pp2mp_offset: origin xyz=1.722275552576525e-17 2.4110002110676104e-17 -3.2175644141916336e-17 rpy=0.0 0.0 0.0 -> xyz=1.9461750163187066e-17 3.195966925249782e-17 5.1027793401258624e-17 rpy=0.0 0.0 0.0
- joint middle_mp2dp: axis -0.9999999999999994 1.159735553967606e-16 6.744138602805412e-17 -> -1.0000000000000002 -3.2838929933875956e-17 5.315090385248316e-16; origin xyz=0.0010000000000000631 9.161508357502633e-18 0.028000000000000025 rpy=1.5707963267948948 0.0 1.5707963267948966 -> xyz=0.0010000000000037676 -2.2551405187698492e-17 0.027999999999999955 rpy=4.551914400963142e-14 -4.440892098500626e-16 1.5707963267948966
- joint middle_mp2dp_offset: origin xyz=-1.5612511283791412e-17 1.3361333028928368e-19 -1.2273161319545561e-16 rpy=0.0 0.0 0.0 -> xyz=-0.011000000000000034 7.28147046937894e-06 0.009007281470469267 rpy=0.0 0.0 0.0
- joint pinky_mp2dp: axis -1.0000000000000002 -3.0531133177191805e-16 -7.355227538141662e-16 -> -0.9999999999999996 2.3037127760972e-15 1.584097436557741e-13; origin xyz=0.0009999999999999842 6.46455545344482e-18 0.028000000000000067 rpy=1.570796326794896 4.440892098500626e-16 1.5707963267948968 -> xyz=0.0010000000000103548 -1.148039996401451e-14 0.02799999999999978 rpy=1.7696955012524995e-13 -1.5853984791647235e-13 1.5707963267948981
- joint pinky_mp2dp_offset: origin xyz=-0.00010000000000001497 -7.207742161365743e-17 -2.9290399316053706e-18 rpy=0.0 0.0 0.0 -> xyz=-0.011000000000000044 7.281470469290411e-06 0.00900728147046922 rpy=0.0 0.0 0.0
- joint ring_abd: axis 6.38378239159465e-16 7.771561172376096e-16 0.9999999999999978 -> -8.004708007547379e-14 -1.9984014443252818e-14 0.9999999999999978; origin xyz=0.019694864162417412 0.0013825982229840389 0.030586364349873878 rpy=-1.5707963267948921 1.3088618425821554 -3.054326190990074 -> xyz=0.019694864162417412 0.0013825982229840321 0.030586364349873787 rpy=-1.5707963267948921 1.3088618425821554 -3.054326190990074
- joint ring_abd_offset: origin xyz=-0.014399999999999944 5.941427905220564e-17 1.5178830414797062e-17 rpy=0.0 0.0 0.0 -> xyz=-0.014400000000000029 3.5561831257524545e-17 8.239936510889834e-18 rpy=0.0 0.0 0.0
- joint ring_mp2dp: axis -1.0000000000000004 -8.881784197001252e-16 9.020562075079397e-17 -> -1.0000000000000004 9.71445146547012e-17 4.7009379895712744e-15; origin xyz=0.0010000000000000406 1.4632114375292307e-16 0.028000000000000025 rpy=1.5707963267948963 2.6645352591003757e-15 1.5707963267948963 -> xyz=0.0010000000000000247 1.5785983631388945e-16 0.02800000000000006 rpy=-1.4432899320127035e-15 -2.886579864025407e-15 1.570796326794897
- joint ring_mp2dp_offset: origin xyz=-1.3721384550404466e-16 -6.547177265705249e-17 -4.2773936368871135e-17 rpy=0.0 0.0 0.0 -> xyz=-0.011000000000000136 7.2814704693049395e-06 0.009007281470469263 rpy=0.0 0.0 0.0
- joint ring_pp2mp: axis -2.7755575615628914e-16 -0.9999999999999994 1.734723475976807e-15 -> 5.551115123125783e-17 -0.9999999999999998 1.6514567491299204e-15; origin xyz=-8.020486901317957e-19 8.994390474632575e-17 0.04800000000000009 rpy=-2.465190328815662e-32 -4.440892098500626e-16 1.1102230246251565e-16 -> xyz=1.6557794334752767e-17 1.0283099349852077e-16 0.048000000000000105 rpy=-8.326672684688684e-17 4.440892098500626e-16 -4.440892098500627e-16
- joint ring_pp2mp_offset: origin xyz=-2.4785122580526127e-17 -9.905120299520399e-17 -1.2157278934836427e-17 rpy=0.0 0.0 0.0 -> xyz=-2.4797730845642552e-17 -9.545841872561936e-17 -2.5561932479781495e-17 rpy=0.0 0.0 0.0
- joint root2index_pp: axis 9.992007221626409e-16 -1.000000000000004 -1.0130785099704553e-15 -> 3.175237850427948e-14 -1.0000000000000018 -2.0646956366832114e-12; origin xyz=-6.511929505797567e-17 -1.2884579059542108e-16 1.2330918261215923e-17 rpy=-3.14159265358971 -1.5689140977438238 3.141592653589709 -> xyz=-3.726525911802163e-14 1.5826592868386048e-13 -1.3897728001093473e-14 rpy=3.141592653571369 -1.568914097743692 -3.1415926535734324
- joint root2index_pp_offset: origin xyz=-2.2103198581084714e-18 -7.053339437169385e-18 1.2080891234349761e-18 rpy=0.0 0.0 0.0 -> xyz=9.357535447968366e-19 9.360525909273759e-18 1.2460153634354755e-17 rpy=0.0 0.0 0.0
- joint root2ring_pp: axis -5.551115123125783e-17 -1.0000000000000022 1.7139067942650854e-15 -> 2.1538326677728037e-14 -1.0000000000000016 9.536885170469134e-13; origin xyz=-8.061277083623726e-17 -2.084317473075087e-17 -8.48575991563069e-18 rpy=3.1415926535897474 -1.569095233503671 -3.1415926535897465 -> xyz=8.76421389591046e-16 -6.591883351625457e-14 -5.609920274269105e-15 rpy=3.1415926535778085 -1.5690952335036443 -3.1415926535768572
- joint root2ring_pp_offset: origin xyz=2.763004548120401e-19 6.477168015932836e-18 1.61034059853451e-17 rpy=0.0 0.0 0.0 -> xyz=-9.795286269233676e-19 -1.4465518891423126e-19 1.4329772049885697e-17 rpy=0.0 0.0 0.0
- joint root2tower_fixed: parent hand_root -> root
- joint thumb_mp2dp: axis 0.9999999999999958 -9.992007221626409e-16 1.7486012637846216e-15 -> -0.9999999999999958 2.9976021664879227e-15 5.287437154777308e-15; limit lower=-1.7453292519943295 upper=0.0 effort=100 velocity=100 -> lower=0.0 upper=1.57 effort=100 velocity=100; origin xyz=1.239088163743751e-16 5.408958416957225e-16 0.03000000000000005 rpy=1.5707963267949039 -8.659739592076221e-15 1.570796326794891 -> xyz=1.8258726914308424e-16 5.204170427930421e-16 0.029999999999999895 rpy=2.4424906541753444e-15 -1.2878587085651816e-14 1.5707963267948923
- joint thumb_mp2dp_offset: origin xyz=-6.3846885802101e-17 -2.638575629691531e-17 -2.8715865630147274e-17 rpy=0.0 0.0 0.0 -> xyz=-0.011000000000000175 7.281470469432116e-06 0.009007281470469333 rpy=0.0 0.0 0.0

Commit message: bug fixes viz

File: src/viz/models/orca1_hand/urdf/orca1.urdf (robot description, URDF)
Before this commit: robot converted_robot, 55 links, 54 joints
Links:
- removed link root
- removed link world
- removed link world2root_fixed_jointbody
- added link hand_root, mass 0.0
Joints:
- removed joint world2root_fixed
- removed joint world2root_fixed_offset
- joint root2palm_fixed: parent root -> hand_root

File: src/viz/models/orca2_hand/urdf/orca2.urdf (robot description, URDF)
Before this commit: robot converted_robot, 57 links, 56 joints
Links:
- removed link root
- removed link world
- removed link world2root_fixed_jointbody
- added link hand_root, mass 0.0
Joints:
- removed joint world2root_fixed
- removed joint world2root_fixed_offset
- joint root2tower_fixed: parent root -> hand_root
