Commit message: fingertip positioning fixes

File: src/viz/models/orca1_hand/urdf/orca1.urdf (robot description, URDF)
Before this commit: robot converted_robot, 53 links, 52 joints
Joints:
- joint index_dp2index_fingertip_fixed: origin xyz=0.0 0.02 -0.001306 rpy=0.0 0.0 0.0 -> xyz=0.011 0.0 0.022 rpy=0.0 0.0 0.0
- joint middle_dp2middle_fingertip_fixed: origin xyz=0.0 0.02 -0.001306 rpy=0.0 0.0 0.0 -> xyz=0.011 0.0 0.022 rpy=0.0 0.0 0.0
- joint pinky_dp2pinky_fingertip_fixed: origin xyz=0.0 0.02 -0.001306 rpy=0.0 0.0 0.0 -> xyz=0.011 0.0 0.022 rpy=0.0 0.0 0.0
- joint ring_dp2ring_fingertip_fixed: origin xyz=0.0 0.02 -0.001306 rpy=0.0 0.0 0.0 -> xyz=0.011 0.0 0.022 rpy=0.0 0.0 0.0
- joint thumb_dp2thumb_fingertip_fixed: origin xyz=0.0 0.02425 -0.001189 rpy=0.0 0.0 0.0 -> xyz=0.011 0.0 0.022 rpy=0.0 0.0 0.0

File: src/viz/models/orca2_hand/urdf/orca2.urdf (robot description, URDF)
Before this commit: robot converted_robot, 55 links, 54 joints
Joints:
- joint index_dp2index_fingertip_fixed: origin xyz=0.0 0.02 -0.001306 rpy=0.0 0.0 0.0 -> xyz=0.011 0.0 0.022 rpy=0.0 0.0 0.0
- joint middle_dp2middle_fingertip_fixed: origin xyz=0.0 0.02 -0.001306 rpy=0.0 0.0 0.0 -> xyz=0.011 0.0 0.022 rpy=0.0 0.0 0.0
- joint pinky_dp2pinky_fingertip_fixed: origin xyz=0.0 0.02 -0.001306 rpy=0.0 0.0 0.0 -> xyz=0.011 0.0 0.022 rpy=0.0 0.0 0.0
- joint ring_dp2ring_fingertip_fixed: origin xyz=0.0 0.02 -0.001306 rpy=0.0 0.0 0.0 -> xyz=0.011 0.0 0.022 rpy=0.0 0.0 0.0
- joint thumb_dp2thumb_fingertip_fixed: origin xyz=0.0 0.02425 -0.001189 rpy=0.0 0.0 0.0 -> xyz=0.011 0.0 0.022 rpy=0.0 0.0 0.0
